Commit message: "Added sim files"

File: articubot/description/bot_core.xacro (robot description, xacro)
@@ -4,4 +4,7 @@
     <material name = "white">
         <color rgba="1 1 1 1"/>
+    </material>
+    <material name = "orange">
+        <color rgba="1 0.3 0.1 1"/>
     </material>
     <material name = "black">
@@ -12,7 +15,9 @@
     </material>
     <!-- Basic size: 0.3m by 0.3m by 0.15; wheel size: ;  -->
-    <!-- CHASSIS -->
+    <!--BASE LINK -->
+    <!-- ideally between the center of the two drive wheels for differential drive -->
     <link name='base_link'>
     </link>
+    <!-- CHASSIS -->
     <link name = 'chassis'>
         <visual>
@@ -29,12 +34,15 @@
             </geometry>
         </collision>
+        <xacro:inertial_box mass="0.5" x="0.3" y="0.3" z="0.15">
+            <origin xyz="0.15 0 0.075" rpy="0 0 0"/>
+        </xacro:inertial_box>
     </link>
     <joint name="chassis_joint" type="fixed">
         <parent link="base_link" />
-        <parent link="chassis" />
-        <origin xyz="-0.1, 0, 0" />
+        <child link="chassis" />
+        <origin xyz="-0.1 0 0" />
     </joint>
     <!-- LEFT WHEEL -->
-    <joint name = "left_wheel_joint">
+    <joint name = "left_wheel_joint" type="continuous">
         <parent link="base_link"/>
         <child link="left_wheel"/>
@@ -54,10 +62,13 @@
             </geometry>
         </collision>
+        <xacro:inertial_cylinder mass="0.5" length="0.04" radius="0.05">
+            <origin xyz="0 0 0" rpy="0 0 0"/>
+        </xacro:inertial_cylinder>
     </link>
     <!-- RIGHT WHEEL -->
-    <joint name = "right_wheel_joint">
+    <joint name = "right_wheel_joint" type="continuous">
         <parent link="base_link"/>
         <child link="right_wheel"/>
-        <origin xyz="0 0.175 0" rpy="${pi/2} 0 0"/>
+        <origin xyz="0 -0.175 0" rpy="${pi/2} 0 0"/>
         <axis xyz="0 0 -1"/> <!-- rotation direction -->
     </joint>
@@ -74,7 +85,10 @@
             </geometry>
         </collision>
+        <xacro:inertial_cylinder mass="0.5" length="0.04" radius="0.05">
+            <origin xyz="0 0 0" rpy="0 0 0"/>
+        </xacro:inertial_cylinder>
     </link>
     <!-- CASTER WHEEL -->
-    <joint name = "caster_wheel_joint">
+    <joint name = "caster_wheel_joint" type="fixed">
         <parent link="chassis"/>
         <child link="caster_wheel"/>
@@ -86,5 +100,5 @@
                 <sphere radius="0.05"/>
             </geometry>
-            <material name="blue"/>
+            <material name="orange"/>
         </visual>
         <collision>
@@ -93,4 +107,7 @@
             </geometry>
         </collision>
+        <xacro:inertial_sphere mass="0.1" radius="0.05">
+            <origin xyz="0 0 0" rpy="0 0 0"/>
+        </xacro:inertial_sphere>
     </link>
 </robot>
